Commit message: Added Create_1 and updated Dragger URDFs

File: urdf/dragger.urdf (robot description, URDF)
Before this commit: robot robot, 11 links, 10 joints
Links:
- removed link caster_wheel
- removed link chassis
- removed link face_link
- removed link laser_frame
- added link chassis_link, mass 0.5; collision box size=0.9 0.4 0.5; visual box size=0.405 0.38 0.25
- added link gps_link; collision cylinder length=0.04 radius=0.05; visual cylinder length=0.02 radius=0.05
- added link laser_link, mass 0.1; collision cylinder length=0.04 radius=0.05; visual cylinder length=0.04 radius=0.05
- added link left_caster_wheel, mass 0.3; collision cylinder length=0.05 radius=0.12; visual box size=0.06 0.06 0.05500000000000001
- added link right_caster_wheel, mass 0.3; collision cylinder length=0.05 radius=0.12; visual box size=0.06 0.06 0.05500000000000001
- link base_footprint: geometry visual box size=0.9 0.4 0.02
- link base_link: geometry visual sphere radius=0.03
- link imu_link: geometry visual box size=0.1 0.1 0.1
- link left_wheel: mass 0.05 -> 1.0; geometry collision cylinder length=0.09 radius=0.192; visual box size=0.038400000000000004 0.0576 0.099
- link right_wheel: mass 0.05 -> 1.0; geometry collision cylinder length=0.09 radius=0.192; visual box size=0.038400000000000004 0.0576 0.099
Joints:
- removed joint caster_wheel_joint
- removed joint face_joint
- added joint gps_joint: type fixed, parent chassis_link, child gps_link, origin xyz=0.05 0 0.65 rpy=0 0 3.1459
- added joint left_caster_wheel_joint: type continuous, parent chassis_link, child left_caster_wheel, origin xyz=-0.32 0.27 -0.062 rpy=1.5707963267948966 0 0, axis 0 0 1
- added joint right_caster_wheel_joint: type continuous, parent chassis_link, child right_caster_wheel, origin xyz=-0.32 -0.27 -0.062 rpy=1.5707963267948966 0 0, axis 0 0 -1
- joint camera_joint: origin xyz=0.276 0 0.181 rpy=0 0.18 0 -> xyz=0.41000000000000003 0 0.55 rpy=0 0.18 0; parent chassis -> chassis_link
- joint camera_optical_joint: origin xyz=0 0 0 rpy=-1.5707963267948966 0 -1.5707963267948966 -> xyz=0 0 0 rpy=0 0 0
- joint chassis_joint: child chassis -> chassis_link; origin xyz=-0.226 0 -0.01 -> xyz=-0.248 0 -0.01
- joint imu_joint: origin xyz=0 0 0.01 -> xyz=0.248 0 0.04 rpy=0 0 0; parent chassis -> chassis_link
- joint laser_joint: child laser_frame -> laser_link; origin xyz=0.122 0 0.212 rpy=0 0 3.1459 -> xyz=0.275 0 0.57 rpy=0 0 3.1459; parent chassis -> chassis_link
- joint left_wheel_joint: origin xyz=0 0.290 0 rpy=-1.5707963267948966 0 0 -> xyz=0.248 0.29 0 rpy=-1.5707963267948966 0 0; parent base_link -> chassis_link
- joint right_wheel_joint: origin xyz=0 -0.290 0 rpy=1.5707963267948966 0 0 -> xyz=0.248 -0.29 0 rpy=1.5707963267948966 0 0; parent base_link -> chassis_link
